File: kicad/main.kicad_sch (KiCad schematic)
At the start: 35 parts, among them J1 Barrel_Jack, SW1 SW_Push, SW2 UP, SW3 DOWN, SW4 LEFT, SW5 RIGHT, SW6 A, SW7 B, U1 CPU, U2 RAM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

Commit message: Cleanup board, add mounting holes
Parts:
- added D1: RESET, LED_THT:LED_D3.0mm, symbol Device:LED
- added D2: POWER, LED_THT:LED_D3.0mm, symbol Device:LED
- added H1, H2, H3, H4: MountingHole, footprints:Hole_3.5x5, symbol Mechanical:MountingHole
- added J2: Conn, Connector_PinHeader_2.54mm:PinHeader_1x16_P2.54mm_Vertical, symbol Connector:Conn_01x16_Pin
- added R12, R13: 10K, Resistor_THT:R_Axial_DIN0207_L6.3mm_D2.5mm_P10.16mm_Horizontal, symbol Device:R
- SW1: value SW_Push -> RESET
- U6: value 74LS138 -> 74HC138
- X1: value CXO_DIP14 -> 1 MHz
Connections:
- net +5V: now also D2.2 (A)
- net A14: no longer U2.3 (A14), U3.27 (A14)
- net A15: no longer U2.31 (A15), U3.1 (A15)
- net CLOCK: now also J2.10 (Pin_10)
- net D0: now also J2.1 (Pin_1)
- net D1: now also J2.2 (Pin_2)
- net D2: now also J2.3 (Pin_3)
- net D3: now also J2.4 (Pin_4)
- net D4: now also J2.5 (Pin_5)
- net D5: now also J2.6 (Pin_6)
- net D6: now also J2.7 (Pin_7)
- net D7: now also J2.8 (Pin_8)
- net GND: now also U2.3 (A14), U2.31 (A15), U3.1 (A15), U3.27 (A14), J2.16 (Pin_16), R12.1, R13.1
- net LCD: now also J2.14 (Pin_14)
- net R/~{W}: now also J2.11 (Pin_11)
- net ~{INPUT}: now also J2.13 (Pin_13)
- net ~{RAM}: now also J2.12 (Pin_12)
- net ~{RES}: now also D1.2 (A), J2.9 (Pin_9)
- net ~{ROM}: now also J2.15 (Pin_15)
- new net: D2.1 (K), R13.2
- new net: D1.1 (K), R12.2
Other:
- note added: "Індикатори"
- note added: "Тестування"
- moved on the sheet: SW1, U4

Commit message: Add images
Other:
- company: (none) -> Андерсон (https://www.youtube.com/@space.caveman)
- title: (none) -> CaveBoard
Changed lines of the file:
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@@
 (kicad_sch (version 20230121) (generator eeschema)
   (paper "A3")
+  (title_block
+    (title "CaveBoard")
+    (date "2023-12-16")
+    (rev "v1")
+    (company "Андерсон (https://www.youtube.com/@space.caveman)")
+  )
   (junction (at 334.01 215.9) (diameter 0) (color 0 0 0 0)
   )
